File: pillcase36/pillcase36.sch (KiCad schematic (older format))
At the start: 106 parts, among them J1 AudioJack4_Ground, SW1 SW_Push, SW10 SW_Push, SW11 SW_Push, SW12 SW_Push, SW13 SW_Push, SW14 SW_Push, SW15 SW_Push, SW16 SW_Push, SW17 SW_Push, SW18 SW_Push, SW19 SW_Push, SW2 SW_Push, SW20 SW_Push, SW21 SW_Push, SW22 SW_Push, SW23 SW_Push, SW24 SW_Push, SW25 SW_Push, SW26 SW_Push, SW27 SW_Push, SW28 SW_Push, SW29 SW_Push, SW3 SW_Push, SW30 SW_Push, SW31 SW_Push, SW32 SW_Push, SW33 SW_Push, SW34 SW_Push, SW35 SW_Push, SW36 SW_Push, SW37 SW_Push, SW4 SW_Push, SW5 SW_Push, SW6 SW_Push, SW7 SW_Push, SW8 SW_Push, SW9 SW_Push, U1 BlackPill, U2 24LC00

Commit message: add PCB
Parts:
- added JP13, JP14: SolderJumper_2_Bridged, pillcase36:JP, symbol Jumper:SolderJumper_2_Bridged
- added TP1: B13, Measurement_Points:Measurement_Point_Round-TH_Small, symbol Connector:TestPoint
- added TP15: B7, Measurement_Points:Measurement_Point_Round-TH_Small, symbol Connector:TestPoint
- added TP16: B11, Measurement_Points:Measurement_Point_Round-TH_Small, symbol Connector:TestPoint
- added TP19: A5, Measurement_Points:Measurement_Point_Round-TH_Small, symbol Connector:TestPoint
- added TP2: B15, Measurement_Points:Measurement_Point_Round-TH_Small, symbol Connector:TestPoint
- added TP20: A3, Measurement_Points:Measurement_Point_Round-TH_Small, symbol Connector:TestPoint
- added TP21: A1, Measurement_Points:Measurement_Point_Round-TH_Small, symbol Connector:TestPoint
- added TP24: B10, Measurement_Points:Measurement_Point_Round-TH_Small, symbol Connector:TestPoint
- added TP27: A4, Measurement_Points:Measurement_Point_Round-TH_Small, symbol Connector:TestPoint
- added TP28: A2, Measurement_Points:Measurement_Point_Round-TH_Small, symbol Connector:TestPoint
- added TP29: A0, Measurement_Points:Measurement_Point_Round-TH_Small, symbol Connector:TestPoint
- added TP31: R1, Measurement_Points:Measurement_Point_Round-TH_Small, symbol Connector:TestPoint
- added TP32: R2, Measurement_Points:Measurement_Point_Round-TH_Small, symbol Connector:TestPoint
- added TP7: B6, Measurement_Points:Measurement_Point_Round-TH_Small, symbol Connector:TestPoint
- added TP8: B12, Measurement_Points:Measurement_Point_Round-TH_Small, symbol Connector:TestPoint
- added TP9: B14, Measurement_Points:Measurement_Point_Round-TH_Small, symbol Connector:TestPoint
- D1, D10, D11, D12, D13, D14, D15, D16, D17, D18, D19, D2, D20, D21, D22, D23, D24, D25, D26, D27, D28, D29, D3, D30, D31, D32, D33, D34, D35, D36, D4, D5, D6, D7, D8, D9: footprint (none) -> pillcase36:Diode_SMD_THT_N
- J1: footprint (none) -> pillcase36:trrs_jack_aki_flip
- JP1, JP10, JP11, JP12, JP2, JP3, JP4, JP5, JP6, JP7, JP8, JP9: footprint (none) -> pillcase36:JP
- R1, R2: footprint (none) -> pillcase36:Resister_SMD_THT_N
- SW1, SW10, SW11, SW12, SW13, SW14, SW15, SW16, SW17, SW18, SW19, SW2, SW20, SW21, SW22, SW23, SW24, SW25, SW26, SW27, SW28, SW29, SW3, SW30, SW31, SW32, SW33, SW34, SW35, SW36, SW4, SW5, SW6, SW7, SW8, SW9: footprint (none) -> pillcase36:key_switch_mx
- SW37: footprint (none) -> Buttons_Switches_THT:SW_PUSH_6mm_h5mm
- TP10: renamed from TP5; footprint (none) -> Measurement_Points:Measurement_Point_Round-TH_Small
- TP11: renamed from TP6; footprint (none) -> Measurement_Points:Measurement_Point_Round-TH_Small
- TP12: renamed from TP7; footprint (none) -> Measurement_Points:Measurement_Point_Round-TH_Small
- TP13: renamed from TP8; footprint (none) -> Measurement_Points:Measurement_Point_Round-TH_Small
- TP14: renamed from TP9; footprint (none) -> Measurement_Points:Measurement_Point_Round-TH_Small
- TP17: renamed from TP10; footprint (none) -> Measurement_Points:Measurement_Point_Round-TH_Small
- TP18: renamed from TP11; footprint (none) -> Measurement_Points:Measurement_Point_Round-TH_Small
- TP22: renamed from TP12; footprint (none) -> Measurement_Points:Measurement_Point_Round-TH_Small
- TP23: renamed from TP13; footprint (none) -> Measurement_Points:Measurement_Point_Round-TH_Small
- TP25: renamed from TP14; footprint (none) -> Measurement_Points:Measurement_Point_Round-TH_Small
- TP26: renamed from TP15; footprint (none) -> Measurement_Points:Measurement_Point_Round-TH_Small
- TP3: renamed from TP1; footprint (none) -> Measurement_Points:Measurement_Point_Round-TH_Small
- TP30: renamed from TP16; footprint (none) -> Measurement_Points:Measurement_Point_Round-TH_Small
- TP4: renamed from TP2; footprint (none) -> Measurement_Points:Measurement_Point_Round-TH_Small
- TP5: renamed from TP3; footprint (none) -> Measurement_Points:Measurement_Point_Round-TH_Small
- TP6: renamed from TP4; footprint (none) -> Measurement_Points:Measurement_Point_Round-TH_Small
- U1: footprint (none) -> pillcase36:BlackPill
- U2: footprint (none) -> SMD_Packages:SOIC-8-N
Connections:
- wire segments 299 -> 323

Commit message: main_v1.0 release
Parts:
- removed JP1, JP10, JP11, JP12, JP2, JP3, JP4, JP5, JP6, JP7, JP8, JP9: SolderJumper_2_Bridged, pillcase36:JP, symbol Jumper:SolderJumper_2_Bridged
- added 0.1u1: C, Capacitors_SMD:C_0603, symbol Device:C
Connections:
- wire segments 323 -> 315
Changed lines of the file:
@@
-$EndComp
-$Comp
-L Jumper:SolderJumper_2_Bridged JP1
-U 1 1 5B83F1CB
-P 1750 2350
-F 0 "JP1" H 1750 2555 50  0000 C CNN
-F 1 "SolderJumper_2_Bridged" H 1750 2464 50  0000 C CNN
-F 2 "pillcase36:JP" H 1750 2350 50  0001 C CNN
-F 3 "~" H 1750 2350 50  0001 C CNN
-	1    1750 2350
-	1    0    0    -1
 $EndComp
 $Comp
@@
 	2000 1900 2050 1900
 Wire Wire Line
-	2000 1550 2000 1900
-Wire Wire Line
 	2450 1900 2550 1900
 Wire Wire Line
 	2550 1900 2550 2000
 Connection ~ 2000 1900
-Wire Wire Line
-	1900 2350 2550 2350
 Wire Wire Line
 	2550 2350 2550 2300
@@
 	2750 1900 2800 1900
 Wire Wire Line
-	2750 1550 2750 1900
-Wire Wire Line
 	3200 1900 3300 1900
 Wire Wire Line
@@
 	3500 1900 3550 1900
 Wire Wire Line
-	3500 1550 3500 1900
-Wire Wire Line
 	3950 1900 4050 1900
 Wire Wire Line
@@
 	4250 1900 4300 1900
 Wire Wire Line
-	4250 1550 4250 1900
-Wire Wire Line
 	4700 1900 4800 1900
 Wire Wire Line
@@
 	5000 1900 5050 1900
 Wire Wire Line
-	5000 1550 5000 1900
-Wire Wire Line
 	5450 1900 5550 1900
 Wire Wire Line
@@
 	5750 1900 5800 1900
 Wire Wire Line
-	5750 1550 5750 1900
-Wire Wire Line
 	6200 1900 6300 1900
 Wire Wire Line
@@
 Connection ~ 2000 2800
 Wire Wire Line
-	1900 3250 2550 3250
-Wire Wire Line
 	2550 3250 2550 3200
 Connection ~ 2550 3250
@@
 Connection ~ 2000 3700
 Wire Wire Line
-	1900 4150 2550 4150
-Wire Wire Line
 	2550 4150 2550 4100
 Connection ~ 2550 4150
@@
 Connection ~ 2000 4600
 Wire Wire Line
-	1900 5050 2550 5050
-Wire Wire Line
 	2550 5050 2550 5000
 Connection ~ 2550 5050
@@
 Connection ~ 2000 5500
 Wire Wire Line
-	1900 5950 2550 5950
-Wire Wire Line
 	2550 5950 2550 5900
 Connection ~ 2550 5950
@@
 	2550 6400 2550 6500
 Wire Wire Line
-	1900 6850 2550 6850
-Wire Wire Line
 	2550 6850 2550 6800
 Connection ~ 2550 6850
@@
 	5750 5500 5750 6400
 $Comp
-L Jumper:SolderJumper_2_Bridged JP2
-U 1 1 5B8B7BA8
-P 1750 3250
-F 0 "JP2" H 1750 3455 50  0000 C CNN
-F 1 "SolderJumper_2_Bridged" H 1750 3364 50  0000 C CNN
-F 2 "pillcase36:JP" H 1750 3250 50  0001 C CNN
-F 3 "~" H 1750 3250 50  0001 C CNN
-	1    1750 3250
-	1    0    0    -1
-$EndComp
-$Comp
-L Jumper:SolderJumper_2_Bridged JP3
-U 1 1 5B8C3C18
-P 1750 4150
-F 0 "JP3" H 1750 4355 50  0000 C CNN
-F 1 "SolderJumper_2_Bridged" H 1750 4264 50  0000 C CNN
-F 2 "pillcase36:JP" H 1750 4150 50  0001 C CNN
-F 3 "~" H 1750 4150 50  0001 C CNN
-	1    1750 4150
-	1    0    0    -1
-$EndComp
-$Comp
-L Jumper:SolderJumper_2_Bridged JP4
-U 1 1 5B8CFC97
-P 1750 5050
-F 0 "JP4" H 1750 5255 50  0000 C CNN
-F 1 "SolderJumper_2_Bridged" H 1750 5164 50  0000 C CNN
-F 2 "pillcase36:JP" H 1750 5050 50  0001 C CNN
-F 3 "~" H 1750 5050 50  0001 C CNN
-	1    1750 5050
-	1    0    0    -1
-$EndComp
-$Comp
-L Jumper:SolderJumper_2_Bridged JP5
-U 1 1 5B8DBD1F
-P 1750 5950
-F 0 "JP5" H 1750 6155 50  0000 C CNN
-F 1 "SolderJumper_2_Bridged" H 1750 6064 50  0000 C CNN
-F 2 "pillcase36:JP" H 1750 5950 50  0001 C CNN
-F 3 "~" H 1750 5950 50  0001 C CNN
-	1    1750 5950
-	1    0    0    -1
-$EndComp
-$Comp
-L Jumper:SolderJumper_2_Bridged JP6
-U 1 1 5B8E7DA4
-P 1750 6850
-F 0 "JP6" H 1750 7055 50  0000 C CNN
-F 1 "SolderJumper_2_Bridged" H 1750 6964 50  0000 C CNN
-F 2 "pillcase36:JP" H 1750 6850 50  0001 C CNN
-F 3 "~" H 1750 6850 50  0001 C CNN
-	1    1750 6850
-	1    0    0    -1
-$EndComp
-$Comp
-L Jumper:SolderJumper_2_Bridged JP7
-U 1 1 5B8F3E6D
-P 2000 1400
-F 0 "JP7" H 2000 1605 50  0000 C CNN
-F 1 "SolderJumper_2_Bridged" H 2000 1514 50  0000 C CNN
-F 2 "pillcase36:JP" H 2000 1400 50  0001 C CNN
-F 3 "~" H 2000 1400 50  0001 C CNN
-	1    2000 1400
-	0    1    1    0
-$EndComp
-$Comp
-L Jumper:SolderJumper_2_Bridged JP8
-U 1 1 5B93C255
-P 2750 1400
-F 0 "JP8" H 2750 1605 50  0000 C CNN
-F 1 "SolderJumper_2_Bridged" H 2750 1514 50  0000 C CNN
-F 2 "pillcase36:JP" H 2750 1400 50  0001 C CNN
-F 3 "~" H 2750 1400 50  0001 C CNN
-	1    2750 1400
-	0    1    1    0
-$EndComp
-$Comp
-L Jumper:SolderJumper_2_Bridged JP9
-U 1 1 5B9482DF
-P 3500 1400
-F 0 "JP9" H 3500 1605 50  0000 C CNN
-F 1 "SolderJumper_2_Bridged" H 3500 1514 50  0000 C CNN
-F 2 "pillcase36:JP" H 3500 1400 50  0001 C CNN
-F 3 "~" H 3500 1400 50  0001 C CNN
-	1    3500 1400
-	0    1    1    0
-$EndComp
-$Comp
-L Jumper:SolderJumper_2_Bridged JP10
-U 1 1 5B954366
-P 4250 1400
-F 0 "JP10" H 4250 1605 50  0000 C CNN
-F 1 "SolderJumper_2_Bridged" H 4250 1514 50  0000 C CNN
-F 2 "pillcase36:JP" H 4250 1400 50  0001 C CNN
-F 3 "~" H 4250 1400 50  0001 C CNN
-	1    4250 1400
-	0    1    1    0
-$EndComp
-$Comp
-L Jumper:SolderJumper_2_Bridged JP11
-U 1 1 5B9603F6
-P 5000 1400
-F 0 "JP11" H 5000 1605 50  0000 C CNN
-F 1 "SolderJumper_2_Bridged" H 5000 1514 50  0000 C CNN
-F 2 "pillcase36:JP" H 5000 1400 50  0001 C CNN
-F 3 "~" H 5000 1400 50  0001 C CNN
-	1    5000 1400
-	0    1    1    0
-$EndComp
-$Comp
-L Jumper:SolderJumper_2_Bridged JP12
-U 1 1 5B96C46F
-P 5750 1400
-F 0 "JP12" H 5750 1605 50  0000 C CNN
-F 1 "SolderJumper_2_Bridged" H 5750 1514 50  0000 C CNN
-F 2 "pillcase36:JP" H 5750 1400 50  0001 C CNN
-F 3 "~" H 5750 1400 50  0001 C CNN
-	1    5750 1400
-	0    1    1    0
-$EndComp
-$Comp
 L Memory_EEPROM:24LC00 U2
 U 1 1 5B9A9C53
@@
 Text GLabel 7450 2800 0    50   Input ~ 0
 SDA1
-Text GLabel 1400 2350 0    50   Input ~ 0
+Text GLabel 1700 2350 0    50   Input ~ 0
 ROW0
-Text GLabel 1400 3250 0    50   Input ~ 0
+Text GLabel 1700 3250 0    50   Input ~ 0
 ROW1
-Text GLabel 1400 4150 0    50   Input ~ 0
+Text GLabel 1700 4150 0    50   Input ~ 0
 ROW2
-Text GLabel 1400 5050 0    50   Input ~ 0
+Text GLabel 1700 5050 0    50   Input ~ 0
 ROW3
-Text GLabel 1400 5950 0    50   Input ~ 0
+Text GLabel 1700 5950 0    50   Input ~ 0
 ROW4
-Text GLabel 1400 6850 0    50   Input ~ 0
+Text GLabel 1700 6850 0    50   Input ~ 0
 ROW5
-Wire Wire Line
-	1400 2350 1600 2350
-Wire Wire Line
-	1400 3250 1600 3250
-Wire Wire Line
-	1400 4150 1600 4150
-Wire Wire Line
-	1400 5050 1600 5050
-Wire Wire Line
-	1600 5950 1400 5950
-Wire Wire Line
-	1400 6850 1600 6850
-Text GLabel 2000 1050 1    50   Input ~ 0
+Text GLabel 2000 1350 1    50   Input ~ 0
 COL0
-Text GLabel 2750 1050 1    50   Input ~ 0
+Text GLabel 2750 1350 1    50   Input ~ 0
 COL1
-Text GLabel 3500 1050 1    50   Input ~ 0
+Text GLabel 3500 1350 1    50   Input ~ 0
 COL2
-Text GLabel 4250 1050 1    50   Input ~ 0
+Text GLabel 4250 1350 1    50   Input ~ 0
 COL3
-Text GLabel 5000 1050 1    50   Input ~ 0
+Text GLabel 5000 1350 1    50   Input ~ 0
 COL4
-Text GLabel 5750 1050 1    50   Input ~ 0
+Text GLabel 5750 1350 1    50   Input ~ 0
 COL5
-Wire Wire Line
-	2000 1050 2000 1250
-Wire Wire Line
-	2750 1050 2750 1250
-Wire Wire Line
-	3500 1050 3500 1250
-Wire Wire Line
-	4250 1050 4250 1250
-Wire Wire Line
-	5000 1050 5000 1250
-Wire Wire Line
-	5750 1050 5750 1250
 Text GLabel 10700 4150 2    50   Input ~ 0
 SDA1
@@
 	8500 5700 8500 5850
 Connection ~ 8500 5850
+Wire Wire Line
+	1700 2350 2550 2350
+Wire Wire Line
+	1700 3250 2550 3250
+Wire Wire Line
+	1700 4150 2550 4150
+Wire Wire Line
+	1700 5050 2550 5050
+Wire Wire Line
+	1700 5950 2550 5950
+Wire Wire Line
+	1700 6850 2550 6850
+Wire Wire Line
+	2000 1350 2000 1900
+Wire Wire Line
+	2750 1350 2750 1900
+Wire Wire Line
+	3500 1350 3500 1900
+Wire Wire Line
+	4250 1350 4250 1900
+Wire Wire Line
+	5000 1350 5000 1900
+Wire Wire Line
+	5750 1350 5750 1900
+$Comp
+L Device:C 0.1u1
+U 1 1 5B911160
+P 9150 4250
+F 0 "0.1u1" H 9265 4296 50  0000 L CNN
+F 1 "C" H 9265 4205 50  0000 L CNN
+F 2 "Capacitors_SMD:C_0603" H 9188 4100 50  0001 C CNN
+F 3 "~" H 9150 4250 50  0001 C CNN
+	1    9150 4250
+	1    0    0    -1
+$EndComp
+Wire Wire Line
+	9150 4100 9150 3850
+Wire Wire Line
+	9150 3850 10000 3850
+Wire Wire Line
+	9150 4400 9150 4600
+Wire Wire Line
+	9150 4600 9450 4600
+Connection ~ 9450 4600
 $EndSCHEMATC
