File: pillcase36/pillcase36.kicad_pcb (KiCad board)
At the start: 2 copper layers, 114 x 140.5 mm, 116 parts, among them J1 AudioJack4_Ground, SW1 SW_Push, SW10 SW_Push, SW11 SW_Push, SW12 SW_Push, SW13 SW_Push, SW14 SW_Push, SW15 SW_Push, SW16 SW_Push, SW17 SW_Push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

Commit message: PCB v1.0.1 Release
Other:
- board text added: "PILLCASE36 v1.0 @Pekaso 2018 Self-Made Keyboards in Japan Discord Group"
- board text removed: "PILLCASE36 v1.0 @Pekaso 2018 Self-Made Keyboards in Japan Dicord Group"
